File: hardware/pomodorov2.kicad_sch (KiCad schematic)
At the start: 12 parts, among them J1 USB_B_Micro, J2 TC2050-IDC, J3 SOICbite, U1 MDBT50Q-1MV2, Y1 32.768kHz

Commit message: Remove SOICBite (for now?)
Parts:
- removed J3: SOICbite, SOICbite:SOIC_clipProgSmall, symbol Connector_Generic:Conn_01x08
Connections:
- no-connect marks 6 -> 4
Other:
- note added: "Pomodoro Timer V2 (Codename: "Otter")"
- note removed: "Pomodoro Timer V2"
- note removed: "SOICbite debug header"
- moved on the sheet: J1, J2, R1, R2, TP1, TP2
